File: hardware/snes_fpc/snes_fpc.kicad_pcb (KiCad board)
At the start: 2 copper layers, 46.6 x 47.5 mm, 7 parts, among them J2 Connector_Generic:Conn_02x16_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, U1 74HC175, U2 74HC4078, U3 74AHC1G08, U4 74AHC1G08

Commit message: Wire missing pads
Parts:
- added J4: Conn_01x02_Pin, Library:Controller_Pads, F.Cu at (87.6, 72.4)
- moved J3 4.35 mm to (91.8, 66.9), turned to -90 degrees
Connections:
- J2 pad 1: AUD_CLK -> BCK
- J2 pad 25: unconnected-(J2-Pin_25-Pad25) -> AUX_1
- J2 pad 26: unconnected-(J2-Pin_26-Pad26) -> AUX_2
- J2 pad 3: AUD_DAT -> LR
- J2 pad 5: AUD_WS -> DAT
- J3 pad 1: unconnected-(J3-BCK-Pad1) -> BCK
- J3 pad 2: unconnected-(J3-DAT-Pad2) -> LR
- J3 pad 3: unconnected-(J3-WS-Pad3) -> DAT
Routing:
- net BRT3: track 2.07 -> 41.1 mm, vias 1 -> 2
- net BRT2: track 1.94 -> 36.6 mm, vias 1 -> 2
- net BRT1: track 3.26 -> 36.3 mm
- net AUX_1: track 0.00 -> 28.3 mm, vias 0 -> 1
- net AUX_2: track 0.00 -> 26.9 mm, vias 0 -> 1
- net DAT: track 0.00 -> 11.4 mm
- net LR: track 0.00 -> 11.0 mm
- net BCK: track 0.00 -> 7.11 mm
- net TRANSP: track 0.00 -> 7.08 mm
Other:
- board size 46.6 x 47.5 mm -> 34.1 x 45 mm

Commit message: WIP footprint adjust
Connections:
- J1 pad 5: (no net) -> +5V
Routing:
- net +5V: track 0.00 -> 47.3 mm, vias 0 -> 1
- net PWR: track 11.0 -> 0.00 mm
- net ADDR_MATCH: track 16.5 -> 15.8 mm, vias 0 -> 2
- net PA7: track 14.9 -> 15.4 mm, vias 2 -> 0
Other:
- outline, holes or cut-outs redrawn

Commit message: Finish routing
Connections:
- J1 pad 16: (no net) -> GND
- J1 pad 30: PAL -> unconnected-(J1-PALMODE-Pad30)
- J1 pad 93: +5V -> PPU2_5V_EXT
- J1 pad 94: +5V -> PPU2_5V_EXT
- J2 pad 6: PAL -> unconnected-(J2-Pin_6-Pad6)
- J2 pad MP: (no net) -> GND
Routing:
- net PIXEL_VALID: track 0.00 -> 19.0 mm
- net CPU_D2: track 0.00 -> 14.6 mm, vias 0 -> 1
- net CPU_D3: track 0.00 -> 14.1 mm, vias 0 -> 1
- net PWR: track 0.00 -> 10.3 mm
- net GND: track 0.00 -> 9.00 mm, vias 0 -> 13
- net PPU2_5V_EXT: track 0.00 -> 3.58 mm
- net +5V: track 47.3 -> 45.0 mm
- net HBLANK: track 35.3 -> 36.6 mm
- net PCLK: track 47.7 -> 48.7 mm
- net VBLANK: track 36.1 -> 37.0 mm
- net CPU_D0: track 4.67 -> 5.46 mm
- net OVER: track 40.2 -> 41.0 mm
- net PA1: track 3.09 -> 3.80 mm
- net PA0: track 3.09 -> 3.80 mm
- net BRT0: track 39.9 -> 40.6 mm, vias 3 -> 2
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- added copper zone on B.Cu, net GND
- added copper zone on F.Cu, net GND
Other:
- outline, holes or cut-outs redrawn

Commit message: Add dec caps
Parts:
- added C1: C_Small_US, Capacitor_SMD:C_0402_1005Metric, F.Cu at (87.1, 76.6)
- added C2: C_Small_US, Capacitor_SMD:C_0402_1005Metric, F.Cu at (92.0, 76.6)
- added C3: C_Small_US, Capacitor_SMD:C_0402_1005Metric, F.Cu at (87.6, 96.7)
- added C4: C_Small_US, Capacitor_SMD:C_0402_1005Metric, F.Cu at (86.6, 89.2)
- U2: value 74HC4078 -> CD4078B
Connections:
- J2 pad MP: GND -> (no net)
Routing:
- net +5V: track 45.0 -> 53.7 mm
- net GND: track 9.00 -> 8.00 mm

Commit message: update fpc
Parts:
- U2: value CD4078B -> 74HC688; footprint Package_SO:TSSOP-14_4.4x5mm_P0.65mm -> Package_SO:TSSOP-20_4.4x6.5mm_P0.65mm
- U3: value 74AHC1G08 -> 74AHC1G32
- moved C3 2.92 mm to (87.2, 99.5)
- moved U2 2.45 mm to (90.2, 95.4)
Connections:
- J2 pad MP: (no net) -> GND
- U2 pad 1: unconnected-(U2-NC-Pad1) -> GND
- U2 pad 10: PA6 -> GND
- U2 pad 11: PA7 -> PA4
- U2 pad 12: unconnected-(U2-NC-Pad12) -> GND
- U2 pad 13: unconnected-(U2-Y-Pad13) -> PA5
- U2 pad 14: +5V -> GND
- U2 pad 3: PA1 -> GND
- U2 pad 4: PA2 -> PA1
- U2 pad 5: PA3 -> GND
- U2 pad 6: PA4 -> PA2
- U2 pad 8: ADDR_MATCH -> PA3
- U2 pad 9: PA5 -> GND
- U3 pad 1: ADDR_MATCH -> ADDR_MATCH_N
Routing:
- net ADDR_MATCH_N: track 0.00 -> 22.3 mm, vias 0 -> 2
- net ADDR_MATCH: track 15.8 -> 0.00 mm, vias 2 -> 0
- net PA4: track 3.09 -> 9.52 mm, vias 0 -> 2
- net +5V: track 53.7 -> 56.8 mm
- net PA0: track 3.80 -> 6.46 mm
- net PA7: track 15.4 -> 17.6 mm
- net PA6: track 10.4 -> 12.4 mm, vias 2 -> 0
- net PCLK: track 48.7 -> 50.5 mm
- net PA1: track 3.80 -> 5.50 mm
- net PA2: track 3.09 -> 4.60 mm
- net VBLANK: track 37.0 -> 38.3 mm
- net HBLANK: track 36.6 -> 37.8 mm
- net PA5: track 9.57 -> 10.7 mm, vias 0 -> 2
- net PA3: track 3.09 -> 4.07 mm
- net BRT3: track 40.7 -> 41.5 mm
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